Commit message: Arm 모델링 링크 수정

File: urdf/so_100_arm_5dof.urdf (robot description, URDF)
Before this commit: robot so_100_arm, 8 links, 7 joints
Links:
- added link gimbal_mount_link; visual mesh filename=package://gimbal_mani/models/gimbal/meshes/gimbal_mount.STL scale=0.001 0.001 0.001
- link Base: geometry collision mesh filename=package://gimbal_mani/models/so_100_arm_5dof/meshes/Base.STL; visual mesh filename=package://gimbal_mani/models/so_100_arm_5dof/meshes/Base.STL
- link Fixed_Gripper: geometry collision mesh filename=package://gimbal_mani/models/so_100_arm_5dof/meshes/Fixed_G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; visual mesh filename=package://gimbal_mani/models/so_100_arm_5dof/meshes/Fixed_G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
- link Lower_Arm: geometry collision mesh filename=package://gimbal_mani/models/so_100_arm_5dof/meshes/Lower_A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; visual mesh filename=package://gimbal_mani/models/so_100_arm_5dof/meshes/Lower_A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
- link Moving_Jaw: geometry collision mesh filename=package://gimbal_mani/models/so_100_arm_5dof/meshes/Moving_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; visual mesh filename=package://gimbal_mani/models/so_100_arm_5dof/meshes/Moving_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
- link Shoulder_Rotation_Pitch: geometry collision mesh filename=package://gimbal_mani/models/so_100_arm_5dof/meshes/Shoulde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; visual mesh filename=package://gimbal_mani/models/so_100_arm_5dof/meshes/Shoulde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
- link Upper_Arm: geometry collision mesh filename=package://gimbal_mani/models/so_100_arm_5dof/meshes/Upper_A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; visual mesh filename=package://gimbal_mani/models/so_100_arm_5dof/meshes/Upper_A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
- link Wrist_Pitch_Roll: geometry collision mesh filename=package://gimbal_mani/models/so_100_arm_5dof/meshes/Wrist_P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; visual mesh filename=package://gimbal_mani/models/so_100_arm_5dof/meshes/Wrist_P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
Joints:
- added joint gimbal_mount_joint: type fixed, parent Fixed_Gripper, child gimbal_mount_link, origin xyz=-0.0155 -0.025 0.0038 rpy=1.6 -1.5708 0

Commit message: ros2_control, 통합 URDF로 이동

File: urdf/so_100_arm_5dof.urdf (robot description, URDF)
Before this commit: robot so_100_arm, 9 links, 8 joints
Joints:
- joint gimbal_mount_joint: origin xyz=-0.0155 -0.025 0.0038 rpy=1.6 -1.5708 0 -> xyz=-0.0171 -0.0263 0.0055 rpy=1.6 -1.5708 0
