Commit message: 오타수정

File: urdf/gimbal_mani.urdf.xacro (robot description, xacro)
@@ -82,5 +82,5 @@
             <state_interface name="velocity"/>
         </joint>
-        <joint name="gimbal_pitch_servo_link">
+        <joint name="gimbal_pitch_servo_joint">
             <command_interface name="position"/>
             <state_interface name="position"/>

Commit message: limits Arm urdf에서 정의

File: urdf/gimbal_mani.urdf.xacro (robot description, xacro)
@@ -24,8 +24,5 @@
         </hardware>
         <joint name="Shoulder_Rotation">
-            <command_interface name="position">
-                <param name="min">-3.14</param>                <!-- todo: 동일 조인트 limit만 보강으로 변경 -->
-                <param name="max">3.14</param>
-            </command_interface>
+            <command_interface name="position"/>
             <state_interface name="position"/>
             <state_interface name="velocity"/>
@@ -33,8 +30,5 @@
         </joint>
         <joint name="Shoulder_Pitch">
-            <command_interface name="position">
-                <param name="min">-3.14</param>
-                <param name="max">3.14</param>
-            </command_interface>
+            <command_interface name="position"/>
             <state_interface name="position"/>
             <state_interface name="velocity"/>
@@ -42,8 +36,5 @@
         </joint>
         <joint name="Elbow">
-            <command_interface name="position">
-                <param name="min">-3.14</param>
-                <param name="max">3.14</param>
-            </command_interface>
+            <command_interface name="position"/>
             <state_interface name="position"/>
             <state_interface name="velocity"/>
@@ -51,8 +42,5 @@
         </joint>
         <joint name="Wrist_Pitch">
-            <command_interface name="position">
-                <param name="min">-3.14</param>
-                <param name="max">3.14</param>
-            </command_interface>
+            <command_interface name="position"/>
             <state_interface name="position"/>
             <state_interface name="velocity"/>
@@ -60,8 +48,5 @@
         </joint>
         <joint name="Wrist_Roll">
-            <command_interface name="position">
-                <param name="min">-3.14</param>
-                <param name="max">3.14</param>
-            </command_interface>
+            <command_interface name="position"/>
             <state_interface name="position"/>
             <state_interface name="velocity"/>
@@ -69,8 +54,5 @@
         </joint>
         <joint name="Gripper">
-            <command_interface name="position">
-                <param name="min">0.0</param>
-                <param name="max">1.57</param>
-            </command_interface>
+            <command_interface name="position"/>
             <state_interface name="position"/>
             <state_interface name="velocity"/>
@@ -88,3 +70,31 @@
         </joint>
     </ros2_control>
+    <gazebo reference="gimbal_camera_link">
+        <sensor name="gimbal_camera" type="camera">
+            <always_on>true</always_on>
+            <update_rate>30</update_rate>
+            <pose>0 0 0 0 0 0</pose>
+            <camera>
+                <horizontal_fov>1.047</horizontal_fov>
+                <image>
+                    <width>640</width>
+                    <height>480</height>
+                    <format>R8G8B8</format>
+                </image>
+                <clip>
+                    <near>0.05</near>
+                    <far>50.0</far>
+                </clip>
+            </camera>
+            <plugin name="gazebo_ros_camera" filename="libgazebo_ros_camera.so">
+                <ros>
+                    <namespace>/gimbal</namespace>
+                </ros>
+                <camera_name>camera</camera_name>
+                <image_topic_name>image_raw</image_topic_name>
+                <camera_info_topic_name>camera_info</camera_info_topic_name>
+                <frame_name>gimbal_camera_link</frame_name>
+            </plugin>
+        </sensor>
+    </gazebo>
 </robot>

File: urdf/so_100_arm_5dof.urdf (robot description, URDF)
Before this commit: robot so_100_arm, 9 links, 8 joints
Joints:
- joint Elbow: limit (none) -> lower=-3.14 upper=3.14 effort=10 velocity=2.0
- joint Gripper: limit (none) -> lower=-3.14 upper=3.14 effort=10 velocity=2.0
- joint Shoulder_Pitch: limit (none) -> lower=-3.14 upper=3.14 effort=10 velocity=2.0
- joint Shoulder_Rotation: limit (none) -> lower=-3.14 upper=3.14 effort=10 velocity=2.0
- joint Wrist_Pitch: limit (none) -> lower=-3.14 upper=3.14 effort=10 velocity=2.0
- joint Wrist_Roll: limit (none) -> lower=-3.14 upper=3.14 effort=10 velocity=2.0

Commit message: 관찰 카메라 위치 이동

File: urdf/gimbal_mani.urdf.xacro (robot description, xacro)
@@ -30,5 +30,5 @@
         <parent link="base_link"/>
         <child link="rear_top_camera_link"/>
-        <origin xyz="-0.8 0.0 0.7" rpy="0.0 0.55 0.0"/>
+        <origin xyz="-0.5 0.4 0.6" rpy="0.0 0.55 -0.75"/>
     </joint>
     <!-- arm -->

Commit message: Gazebo 에서 모델 색 추가

File: urdf/gimbal_mani.urdf.xacro (robot description, xacro)
@@ -2,5 +2,5 @@
 <robot name="gimbal_mani"
     xmlns:xacro="http://www.ros.org/wiki/xacro">
-    <xacro:arg name="mesh_prefix" default=""/>
+    <xacro:arg name="mesh_prefix" default="package://gimbal_mani"/>
     <xacro:property name="mesh_prefix" value="$(arg mesh_prefix)"/>
     <link name="world"/>
@@ -113,4 +113,5 @@
     </ros2_control>
     <gazebo reference="gimbal_camera_link">
+        <material>Gazebo/Black</material>
         <sensor name="gimbal_camera" type="camera">
             <always_on>true</always_on>
@@ -141,8 +142,9 @@
     </gazebo>
     <gazebo reference="tof_link">
+        <material>Gazebo/Red</material>
         <sensor name="tof_ray" type="ray">
             <always_on>true</always_on>
             <update_rate>30</update_rate>
-            <visualize>false</visualize>
+            <visualize>true</visualize>
             <ray>
                 <scan>
