Commit message: 마운트 제외(Arm에 포함)

File: urdf/gimbal.urdf.xacro (robot description, xacro)
@@ -4,17 +4,16 @@
     <!-- ===== params ===== -->
     <xacro:property name="gimbal_pkg" value="gimbal_mani"/>
-    <!-- 패키지명으로 교체 -->
     <xacro:property name="stl_scale" value="0.001 0.001 0.001"/>
     <xacro:property name="yaw_limit" value="3.1416"/>
     <xacro:property name="pitch_limit" value="1.5708"/>
     <!-- ===== root: arm에서 Fixed_Gripper에 붙을 링크 ===== -->
-    <link name="gimbal_mount_link"> <!-- todo: 모델링 수정 -->
+    <!-- <link name="gimbal_mount_link">
         <visual>
             <origin xyz="0 0 0" rpy="0 -1.5707 3.141592"/>
             <geometry>
-                <mesh filename="package://${gimbal_pkg}/models/gimbal/meshes/gimbal_mount.STL" scale="${stl_scale}"/>
+                <mesh filename="package://${gimbal_pkg}/models/gimbal/meshes/gimbal_mount2.stl" scale="${stl_scale}"/>
             </geometry>
         </visual>
-    </link>
+    </link> -->
     <link name="gimbal_base_link">
         <visual>
@@ -25,9 +24,9 @@
         </visual>
     </link>
-    <joint name="gimbal_base_joint" type="fixed">
+    <!-- <joint name="gimbal_base_joint" type="fixed">
         <parent link="gimbal_mount_link"/>
         <child link="gimbal_base_link"/>
         <origin xyz="0.0 0.0 0.0" rpy="0.0 0.0 0.0"/>
-    </joint>
+    </joint> -->
     <link name="gimbal_yaw_servo_link">
         <visual>
@@ -41,7 +40,7 @@
         </visual>
     </link>
-    <joint name="gimbal_yaw_servo_mount_joint" type="revolute">
+    <joint name="gimbal_yaw_servo_joint" type="revolute">
         <parent link="gimbal_base_link"/>
-        <child  link="gimbal_yaw_servo_link"/>
+        <child link="gimbal_yaw_servo_link"/>
         <!-- 서보 축 중심 위치 -->
         <origin xyz="-0.004 0.02 0" rpy="0 0 0"/>
@@ -76,5 +75,5 @@
     <joint name="gimbal_pitch_servo_joint" type="revolute">
         <parent link="gimbal_yaw_link"/>
-        <child  link="gimbal_pitch_servo_link"/>
+        <child link="gimbal_pitch_servo_link"/>
         <!-- 서보 축 중심 위치 -->
         <origin xyz="0.0425 -0.003 0.083" rpy="0 0 0"/>
@@ -82,5 +81,5 @@
         <limit lower="-${pitch_limit}" upper="${pitch_limit}" effort="1.0" velocity="6.0"/>
     </joint>
-    <!-- ===== pitch stage (부품 STL) ===== -->
+    <!-- ===== pitch stage ===== -->
     <link name="gimbal_pitch_link">
         <visual>
@@ -99,6 +98,6 @@
         <limit lower="-${pitch_limit}" upper="${pitch_limit}" effort="1.0" velocity="6.0"/>
     </joint>
-        <!-- ===== camera stage (부품 STL 또는 카메라 STL) ===== -->
-        <!-- <link name="gimbal_camera_link">
+    <!-- ===== camera stage ===== -->
+    <!-- <link name="gimbal_camera_link">
     <visual>
       <origin xyz="0 0 0" rpy="0 0 0"/>
@@ -113,3 +112,3 @@
     <origin xyz="0 0 0" rpy="0 0 0"/>
   </joint> -->
-    </robot>
+</robot>

Commit message: 카메라 정의

File: urdf/gimbal.urdf.xacro (robot description, xacro)
@@ -99,16 +99,9 @@
     </joint>
     <!-- ===== camera stage ===== -->
-    <!-- <link name="gimbal_camera_link">
-    <visual>
-      <origin xyz="0 0 0" rpy="0 0 0"/>
-      <geometry>
-        <mesh filename="package://${gimbal_pkg}/models/gimbal/meshes/camera_part.stl" scale="${stl_scale}"/>
-      </geometry>
-    </visual>
-  </link>
-  <joint name="gimbal_camera_joint" type="fixed">
-    <parent link="gimbal_pitch_link"/>
-    <child link="gimbal_camera_link"/>
-    <origin xyz="0 0 0" rpy="0 0 0"/>
-  </joint> -->
+    <link name="gimbal_camera_link"/>
+    <joint name="gimbal_camera_joint" type="fixed">
+        <parent link="gimbal_pitch_link"/>
+        <child link="gimbal_camera_link"/>
+        <origin xyz="0 0 0" rpy="0 0 0"/>
+    </joint>
 </robot>

Commit message: 메쉬 참조 수정

File: urdf/gimbal.urdf.xacro (robot description, xacro)
@@ -2,6 +2,6 @@
 <robot name="servo_gimbal_2axis"
     xmlns:xacro="http://www.ros.org/wiki/xacro">
+    <xacro:arg name="mesh_prefix" default=""/>
     <!-- ===== params ===== -->
-    <xacro:property name="gimbal_pkg" value="gimbal_mani"/>
     <xacro:property name="stl_scale" value="0.001 0.001 0.001"/>
     <xacro:property name="yaw_limit" value="3.1416"/>
@@ -12,5 +12,5 @@
             <origin xyz="0 0 0" rpy="0 -1.5707 3.141592"/>
             <geometry>
-                <mesh filename="package://${gimbal_pkg}/models/gimbal/meshes/gimbal_mount2.stl" scale="${stl_scale}"/>
+                <mesh filename="${mesh_prefix}/models/gimbal/meshes/gimbal_mount2.stl" scale="${stl_scale}"/>
             </geometry>
         </visual>
@@ -20,5 +20,5 @@
             <origin xyz="-0.5 0.0 0.0225" rpy="0.0 0.0 0.0"/>
             <geometry>
-                <mesh filename="package://${gimbal_pkg}/models/gimbal/meshes/gimbal_base.STL" scale="${stl_scale}"/>
+                <mesh filename="${mesh_prefix}/models/gimbal/meshes/gimbal_base.STL" scale="${stl_scale}"/>
             </geometry>
         </visual>
@@ -53,5 +53,5 @@
             <origin xyz="-0.4965 -0.0188 0.05" rpy="0 0 0"/>
             <geometry>
-                <mesh filename="package://${gimbal_pkg}/models/gimbal/meshes/gimbal_arms.STL" scale="${stl_scale}"/>
+                <mesh filename="${mesh_prefix}/models/gimbal/meshes/gimbal_arms.STL" scale="${stl_scale}"/>
             </geometry>
         </visual>
@@ -86,5 +86,5 @@
             <origin xyz="-0.539 -0.018 -0.0335" rpy="0 0 0"/>
             <geometry>
-                <mesh filename="package://${gimbal_pkg}/models/gimbal/meshes/gimbal_tilt.STL" scale="${stl_scale}"/>
+                <mesh filename="${mesh_prefix}/models/gimbal/meshes/gimbal_tilt.STL" scale="${stl_scale}"/>
             </geometry>
         </visual>

File: urdf/gimbal_mani.urdf.xacro (robot description, xacro)
@@ -2,6 +2,8 @@
 <robot name="gimbal_mani"
     xmlns:xacro="http://www.ros.org/wiki/xacro">
+    <xacro:arg name="mesh_prefix" default=""/>
+    <xacro:property name="mesh_prefix" value="$(arg mesh_prefix)"/>
     <!-- arm -->
-    <xacro:include filename="$(find gimbal_mani)/urdf/so_100_arm_5dof.urdf"/>
+    <xacro:include filename="$(find gimbal_mani)/urdf/so_100_arm_5dof.urdf.xacro"/>
     <!-- gimbal -->
     <xacro:include filename="$(find gimbal_mani)/urdf/gimbal.urdf.xacro"/>

Commit message: 관찰카메라, 초기 pose 설정

File: urdf/gimbal.urdf.xacro (robot description, xacro)
@@ -7,4 +7,12 @@
     <xacro:property name="yaw_limit" value="3.1416"/>
     <xacro:property name="pitch_limit" value="1.5708"/>
+    <xacro:property name="default_mass" value="0.05"/>
+    <xacro:macro name="default_inertial" params="mass">
+        <inertial>
+            <mass value="${mass}"/>
+            <origin xyz="0 0 0" rpy="0 0 0"/>
+            <inertia ixx="1e-5" ixy="0" ixz="0" iyy="1e-5" iyz="0" izz="1e-5"/>
+        </inertial>
+    </xacro:macro>
     <!-- ===== root: arm에서 Fixed_Gripper에 붙을 링크 ===== -->
     <!-- <link name="gimbal_mount_link">
@@ -17,4 +25,5 @@
     </link> -->
     <link name="gimbal_base_link">
+        <xacro:default_inertial mass="${default_mass}"/>
         <visual>
             <origin xyz="-0.5 0.0 0.0225" rpy="0.0 0.0 0.0"/>
@@ -30,4 +39,5 @@
     </joint> -->
     <link name="gimbal_yaw_servo_link">
+        <xacro:default_inertial mass="${default_mass}"/>
         <visual>
             <origin xyz="0.005 0.00 0.048" rpy="0 0 0"/>
@@ -50,4 +60,5 @@
     <!-- ===== yaw stage ===== -->
     <link name="gimbal_yaw_link">
+        <xacro:default_inertial mass="${default_mass}"/>
         <visual>
             <origin xyz="-0.4965 -0.0188 0.05" rpy="0 0 0"/>
@@ -63,4 +74,5 @@
     </joint>
     <link name="gimbal_pitch_servo_link">
+        <xacro:default_inertial mass="${default_mass}"/>
         <visual>
             <origin xyz="0.0 -0.000 0.01" rpy="1.5708 1.5708 0"/>
@@ -83,4 +95,5 @@
     <!-- ===== pitch stage ===== -->
     <link name="gimbal_pitch_link">
+        <xacro:default_inertial mass="${default_mass}"/>
         <visual>
             <origin xyz="-0.539 -0.018 -0.0335" rpy="0 0 0"/>
@@ -99,5 +112,7 @@
     </joint>
     <!-- ===== camera stage ===== -->
-    <link name="gimbal_camera_link"/>
+    <link name="gimbal_camera_link">
+        <xacro:default_inertial mass="0.02"/>
+    </link>
     <joint name="gimbal_camera_joint" type="fixed">
         <parent link="gimbal_pitch_link"/>

File: urdf/gimbal_mani.urdf.xacro (robot description, xacro)
@@ -4,4 +4,32 @@
     <xacro:arg name="mesh_prefix" default=""/>
     <xacro:property name="mesh_prefix" value="$(arg mesh_prefix)"/>
+    <link name="world"/>
+    <joint name="world_to_base" type="fixed">
+        <parent link="world"/>
+        <child link="base_link"/>
+        <origin xyz="0 0 0" rpy="0 0 1.57079632679"/>
+    </joint>
+    <!-- 고정 관찰 카메라 -->
+    <link name="rear_top_camera_link">
+        <inertial>
+            <origin xyz="0 0 0" rpy="0 0 0"/>
+            <mass value="0.01"/>
+            <inertia ixx="1e-6" ixy="0" ixz="0" iyy="1e-6" iyz="0" izz="1e-6"/>
+        </inertial>
+        <visual>
+            <origin xyz="0 0 0" rpy="0 0 0"/>
+            <geometry>
+                <box size="0.02 0.02 0.02"/>
+            </geometry>
+            <material name="rear_cam_marker">
+                <color rgba="1 1 0 1"/>
+            </material>
+        </visual>
+    </link>
+    <joint name="world_to_rear_top_camera" type="fixed">
+        <parent link="base_link"/>
+        <child link="rear_top_camera_link"/>
+        <origin xyz="-0.8 0.0 0.7" rpy="0.0 0.55 0.0"/>
+    </joint>
     <!-- arm -->
     <xacro:include filename="$(find gimbal_mani)/urdf/so_100_arm_5dof.urdf.xacro"/>
@@ -16,16 +44,18 @@
         <origin xyz="0.002 0.004 0" rpy="3.1416 -1.5707 0"/>
     </joint>
-    <plugin filename="gz_ros2_control-system" name="gz_ros2_control::GazeboSimROS2ControlPlugin">
-        <parameters>$(find gimbal_mani)/config/controllers.yaml</parameters>
-        <robot_param>robot_description</robot_param>
-        <robot_param_node>robot_state_publisher</robot_param_node>
-    </plugin>
-    <ros2_control name="gz_ros2_control/GazeboSimSystem" type="system">
+    <gazebo>
+        <plugin filename="libgazebo_ros2_control.so" name="gazebo_ros2_control">
+            <parameters>$(find gimbal_mani)/config/controllers.yaml</parameters>
+        </plugin>
+    </gazebo>
+    <ros2_control name="GazeboSystem" type="system">
         <hardware>
-            <plugin>gz_ros2_control/GazeboSimSystem</plugin>
+            <plugin>gazebo_ros2_control/GazeboSystem</plugin>
         </hardware>
         <joint name="Shoulder_Rotation">
             <command_interface name="position"/>
-            <state_interface name="position"/>
+            <state_interface name="position">
+                <param name="initial_value">0.0</param>
+            </state_interface>
             <state_interface name="velocity"/>
             <state_interface name="effort"/>
@@ -33,5 +63,7 @@
         <joint name="Shoulder_Pitch">
             <command_interface name="position"/>
-            <state_interface name="position"/>
+            <state_interface name="position">
+                <param name="initial_value">-1.5</param>
+            </state_interface>
             <state_interface name="velocity"/>
             <state_interface name="effort"/>
@@ -39,5 +71,7 @@
         <joint name="Elbow">
             <command_interface name="position"/>
-            <state_interface name="position"/>
+            <state_interface name="position">
+                <param name="initial_value">1.5</param>
+            </state_interface>
             <state_interface name="velocity"/>
             <state_interface name="effort"/>
@@ -45,5 +79,7 @@
         <joint name="Wrist_Pitch">
             <command_interface name="position"/>
-            <state_interface name="position"/>
+            <state_interface name="position">
+                <param name="initial_value">-1.5</param>
+            </state_interface>
             <state_interface name="velocity"/>
             <state_interface name="effort"/>
@@ -51,5 +87,7 @@
         <joint name="Wrist_Roll">
             <command_interface name="position"/>
-            <state_interface name="position"/>
+            <state_interface name="position">
+                <param name="initial_value">0.0</param>
+            </state_interface>
             <state_interface name="velocity"/>
             <state_interface name="effort"/>
@@ -57,5 +95,7 @@
         <joint name="Gripper">
             <command_interface name="position"/>
-            <state_interface name="position"/>
+            <state_interface name="position">
+                <param name="initial_value">0.5</param>
+            </state_interface>
             <state_interface name="velocity"/>
             <state_interface name="effort"/>
@@ -100,3 +140,33 @@
         </sensor>
     </gazebo>
+    <gazebo reference="rear_top_camera_link">
+        <sensor name="rear_top_camera" type="camera">
+            <always_on>true</always_on>
+            <update_rate>15</update_rate>
+            <pose>0 0 0 0 0 0</pose>
+            <camera>
+                <horizontal_fov>1.047</horizontal_fov>
+                <image>
+                    <width>640</width>
+                    <height>480</height>
+                    <format>R8G8B8</format>
+                </image>
+                <clip>
+                    <near>0.1</near>
+                    <far>100.0</far>
+                </clip>
+            </camera>
+            <plugin name="gazebo_ros_rear_top_camera" filename="libgazebo_ros_camera.so">
+                <ros>
+                    <namespace>/overview</namespace>
+                    <remapping>image_raw:=/overview/image_raw</remapping>
+                    <remapping>camera_info:=/overview/camera_info</remapping>
+                </ros>
+                <camera_name>rear_top</camera_name>
+                <image_topic_name>image_raw</image_topic_name>
+                <camera_info_topic_name>camera_info</camera_info_topic_name>
+                <frame_name>rear_top_camera_link</frame_name>
+            </plugin>
+        </sensor>
+    </gazebo>
 </robot>

File: urdf/so_100_arm_5dof.urdf.xacro (robot description, xacro)
@@ -13,6 +13,5 @@
     <origin xyz="0 0 0" rpy="0 0 0"/>
   </joint> -->
-  <link
-    name="base_link">
+  <link name="base_link">
     <gazebo>
       <material>Gazebo/Grey</material>
@@ -24,6 +23,5 @@
     <origin xyz="0 0 0" rpy="0 0 0"/>
   </joint>
-  <link
-    name="Base">
+  <link name="Base">
     <inertial>
       <origin

Commit message: ToF 플러그인, 토픽 추가

File: urdf/gimbal.urdf.xacro (robot description, xacro)
@@ -120,3 +120,26 @@
         <origin xyz="0 0 0" rpy="0 0 0"/>
     </joint>
+    <link name="tof_link">
+        <inertial>
+            <origin xyz="0 0 0" rpy="0 0 0"/>
+            <mass value="0.01"/>
+            <inertia ixx="1e-6" ixy="0" ixz="0"
+                     iyy="1e-6" iyz="0"
+                     izz="1e-6"/>
+        </inertial>
+        <visual>
+            <origin xyz="0 0 0" rpy="0 0 0"/>
+            <geometry>
+                <box size="0.02 0.02 0.01"/>
+            </geometry>
+            <material name="tof_visual">
+                <color rgba="0.1 0.8 0.1 1.0"/>
+            </material>
+        </visual>
+    </link>
+    <joint name="tof_joint" type="fixed">
+        <parent link="gimbal_camera_link"/>
+        <child link="tof_link"/>
+        <origin xyz="0.025 0.0 -0.023" rpy="0 0 0"/>
+    </joint>
 </robot>

File: urdf/gimbal_mani.urdf.xacro (robot description, xacro)
@@ -140,4 +140,35 @@
         </sensor>
     </gazebo>
+    <gazebo reference="gimbal_tof_link">
+        <sensor name="tof_ray" type="ray">
+            <always_on>true</always_on>
+            <update_rate>30</update_rate>
+            <visualize>false</visualize>
+            <ray>
+            <scan>
+                <horizontal>
+                <samples>1</samples>
+                <resolution>1</resolution>
+                <min_angle>0</min_angle>
+                <max_angle>0</max_angle>
+                </horizontal>
+            </scan>
+            <range>
+                <min>0.02</min>
+                <max>2.00</max>
+                <resolution>0.001</resolution>
+            </range>
+            </ray>
+        </sensor>
+        <plugin name="tof_controller" filename="libgazebo_ros_ray_sensor.so">
+            <ros>
+            <namespace>/gimbal</namespace>
+            <remapping>~/out:=tof_distance</remapping>
+            </ros>
+            <output_type>sensor_msgs/LaserScan</output_type>
+            <radiation_type>infrared</radiation_type>
+            <frame_name>tof_link</frame_name>
+        </plugin>
+    </gazebo>
     <gazebo reference="rear_top_camera_link">
         <sensor name="rear_top_camera" type="camera">

Commit message: 카메라 형상추가, ToF 위치 변경

File: urdf/gimbal.urdf.xacro (robot description, xacro)
@@ -2,5 +2,5 @@
 <robot name="servo_gimbal_2axis"
     xmlns:xacro="http://www.ros.org/wiki/xacro">
-    <xacro:arg name="mesh_prefix" default=""/>
+    <xacro:arg name="mesh_prefix" default="package://gimbal_mani"/>
     <!-- ===== params ===== -->
     <xacro:property name="stl_scale" value="0.001 0.001 0.001"/>
@@ -29,5 +29,5 @@
             <origin xyz="-0.5 0.0 0.0225" rpy="0.0 0.0 0.0"/>
             <geometry>
-                <mesh filename="${mesh_prefix}/models/gimbal/meshes/gimbal_base.STL" scale="${stl_scale}"/>
+                <mesh filename="${mesh_prefix}/models/gimbal/meshes/gimbal_base.stl" scale="${stl_scale}"/>
             </geometry>
         </visual>
@@ -64,5 +64,5 @@
             <origin xyz="-0.4965 -0.0188 0.05" rpy="0 0 0"/>
             <geometry>
-                <mesh filename="${mesh_prefix}/models/gimbal/meshes/gimbal_arms.STL" scale="${stl_scale}"/>
+                <mesh filename="${mesh_prefix}/models/gimbal/meshes/gimbal_arms.stl" scale="${stl_scale}"/>
             </geometry>
         </visual>
@@ -99,5 +99,5 @@
             <origin xyz="-0.539 -0.018 -0.0335" rpy="0 0 0"/>
             <geometry>
-                <mesh filename="${mesh_prefix}/models/gimbal/meshes/gimbal_tilt.STL" scale="${stl_scale}"/>
+                <mesh filename="${mesh_prefix}/models/gimbal/meshes/gimbal_tilt.stl" scale="${stl_scale}"/>
             </geometry>
         </visual>
@@ -114,9 +114,25 @@
     <link name="gimbal_camera_link">
         <xacro:default_inertial mass="0.02"/>
+        <inertial>
+            <origin xyz="0 0 0" rpy="0 0 0"/>
+            <mass value="0.01"/>
+            <inertia ixx="1e-6" ixy="0" ixz="0"
+                     iyy="1e-6" iyz="0"
+                     izz="1e-6"/>
+        </inertial>
+        <visual>
+            <origin xyz="0 0 0" rpy="0 0 0"/>
+            <geometry>
+                <box size="0.01 0.02 0.02"/>
+            </geometry>
+            <material name="camera_visual">
+                <color rgba="0.6 0.3 0.1 1.0"/>
+            </material>
+        </visual>
     </link>
     <joint name="gimbal_camera_joint" type="fixed">
         <parent link="gimbal_pitch_link"/>
         <child link="gimbal_camera_link"/>
-        <origin xyz="0 0 0" rpy="0 0 0"/>
+        <origin xyz="0.01 0 0.01" rpy="0 0 0"/>
     </joint>
     <link name="tof_link">
@@ -131,5 +147,5 @@
             <origin xyz="0 0 0" rpy="0 0 0"/>
             <geometry>
-                <box size="0.02 0.02 0.01"/>
+                <box size="0.01 0.01 0.01"/>
             </geometry>
             <material name="tof_visual">
@@ -141,5 +157,5 @@
         <parent link="gimbal_camera_link"/>
         <child link="tof_link"/>
-        <origin xyz="0.025 0.0 -0.023" rpy="0 0 0"/>
+        <origin xyz="0 0.01 0" rpy="0 0 0"/>
     </joint>
 </robot>
