Commit message: xacro로 래핑

File: urdf/so_100_arm_5dof.urdf.xacro (robot description, xacro)
@@ -4,30 +4,6 @@
      For more information, please see http://wiki.ros.org/sw_urdf_exporter -->
 <robot
-  name="so_100_arm">
-  <gazebo>
-    <plugin filename="libgz-sim-physics-system.so"
-            name="gz::sim::systems::Physics">
-        <engine>
-            <filename>libgz-physics-ode-plugin.so</filename>
-        </engine>
-        <update_rate>1000</update_rate>
-        <gravity>0 0 -9.8</gravity>
-        <max_step_size>0.001</max_step_size>
-        <real_time_factor>1.0</real_time_factor>
-        <real_time_update_rate>1000</real_time_update_rate>
-        <ode>
-            <solver>
-                <type>quick</type>
-                <iters>50</iters>
-            </solver>
-        </ode>
-    </plugin>
-    <plugin filename="libgz-sim-joint-state-publisher-system.so"
-            name="gz::sim::systems::JointStatePublisher">
-    </plugin>
-    <plugin filename="libgz-sim-pose-publisher-system.so"
-            name="gz::sim::systems::PosePublisher">
-    </plugin>
-  </gazebo>
+  name="so_100_arm" xmlns:xacro="http://www.ros.org/wiki/xacro">
+  <xacro:arg name="mesh_prefix" default=""/>
 <!--
   <link name="world"/>
@@ -70,19 +46,19 @@
       <geometry>
         <mesh
-          filename="package://gimbal_mani/models/so_100_arm_5dof/meshes/Base.STL" />
-      </geometry>
-      <material
-        name="">
-        <color
-          rgba="0.792156862745098 0.819607843137255 0.933333333333333 1" />
-      </material>
-    </visual>
-    <collision>
-      <origin
-        xyz="0 0 0"
-        rpy="0 0 0" />
-      <geometry>
-        <mesh
-          filename="package://gimbal_mani/models/so_100_arm_5dof/meshes/Base.STL" />
+          filename="${mesh_prefix}/models/so_100_arm_5dof/meshes/Base.STL" />
+      </geometry>
+      <material
+        name="">
+        <color
+          rgba="0.792156862745098 0.819607843137255 0.933333333333333 1" />
+      </material>
+    </visual>
+    <collision>
+      <origin
+        xyz="0 0 0"
+        rpy="0 0 0" />
+      <geometry>
+        <mesh
+          filename="${mesh_prefix}/models/so_100_arm_5dof/meshes/Base.STL" />
       </geometry>
     </collision>
@@ -110,19 +86,19 @@
       <geometry>
         <mesh
-          filename="package://gimbal_mani/models/so_100_arm_5dof/meshes/Shoulder_Rotation_Pitch.STL" />
-      </geometry>
-      <material
-        name="">
-        <color
-          rgba="0.792156862745098 0.819607843137255 0.933333333333333 1" />
-      </material>
-    </visual>
-    <collision>
-      <origin
-        xyz="0 0 0"
-        rpy="0 0 0" />
-      <geometry>
-        <mesh
-          filename="package://gimbal_mani/models/so_100_arm_5dof/meshes/Shoulder_Rotation_Pitch.STL" />
+          filename="${mesh_prefix}/models/so_100_arm_5dof/meshes/Shoulder_Rotation_Pitch.STL" />
+      </geometry>
+      <material
+        name="">
+        <color
+          rgba="0.792156862745098 0.819607843137255 0.933333333333333 1" />
+      </material>
+    </visual>
+    <collision>
+      <origin
+        xyz="0 0 0"
+        rpy="0 0 0" />
+      <geometry>
+        <mesh
+          filename="${mesh_prefix}/models/so_100_arm_5dof/meshes/Shoulder_Rotation_Pitch.STL" />
       </geometry>
     </collision>
@@ -164,19 +140,19 @@
       <geometry>
         <mesh
-          filename="package://gimbal_mani/models/so_100_arm_5dof/meshes/Upper_Arm.STL" />
-      </geometry>
-      <material
-        name="">
-        <color
-          rgba="0.792156862745098 0.819607843137255 0.933333333333333 1" />
-      </material>
-    </visual>
-    <collision>
-      <origin
-        xyz="0 0 0"
-        rpy="0 0 0" />
-      <geometry>
-        <mesh
-          filename="package://gimbal_mani/models/so_100_arm_5dof/meshes/Upper_Arm.STL" />
+          filename="${mesh_prefix}/models/so_100_arm_5dof/meshes/Upper_Arm.STL" />
+      </geometry>
+      <material
+        name="">
+        <color
+          rgba="0.792156862745098 0.819607843137255 0.933333333333333 1" />
+      </material>
+    </visual>
+    <collision>
+      <origin
+        xyz="0 0 0"
+        rpy="0 0 0" />
+      <geometry>
+        <mesh
+          filename="${mesh_prefix}/models/so_100_arm_5dof/meshes/Upper_Arm.STL" />
       </geometry>
     </collision>
@@ -218,19 +194,19 @@
       <geometry>
         <mesh
-          filename="package://gimbal_mani/models/so_100_arm_5dof/meshes/Lower_Arm.STL" />
-      </geometry>
-      <material
-        name="">
-        <color
-          rgba="0.792156862745098 0.819607843137255 0.933333333333333 1" />
-      </material>
-    </visual>
-    <collision>
-      <origin
-        xyz="0 0 0"
-        rpy="0 0 0" />
-      <geometry>
-        <mesh
-          filename="package://gimbal_mani/models/so_100_arm_5dof/meshes/Lower_Arm.STL" />
+          filename="${mesh_prefix}/models/so_100_arm_5dof/meshes/Lower_Arm.STL" />
+      </geometry>
+      <material
+        name="">
+        <color
+          rgba="0.792156862745098 0.819607843137255 0.933333333333333 1" />
+      </material>
+    </visual>
+    <collision>
+      <origin
+        xyz="0 0 0"
+        rpy="0 0 0" />
+      <geometry>
+        <mesh
+          filename="${mesh_prefix}/models/so_100_arm_5dof/meshes/Lower_Arm.STL" />
       </geometry>
     </collision>
@@ -272,19 +248,19 @@
       <geometry>
         <mesh
-          filename="package://gimbal_mani/models/so_100_arm_5dof/meshes/Wrist_Pitch_Roll.STL" />
-      </geometry>
-      <material
-        name="">
-        <color
-          rgba="0.792156862745098 0.819607843137255 0.933333333333333 1" />
-      </material>
-    </visual>
-    <collision>
-      <origin
-        xyz="0 0 0"
-        rpy="0 0 0" />
-      <geometry>
-        <mesh
-          filename="package://gimbal_mani/models/so_100_arm_5dof/meshes/Wrist_Pitch_Roll.STL" />
+          filename="${mesh_prefix}/models/so_100_arm_5dof/meshes/Wrist_Pitch_Roll.STL" />
+      </geometry>
+      <material
+        name="">
+        <color
+          rgba="0.792156862745098 0.819607843137255 0.933333333333333 1" />
+      </material>
+    </visual>
+    <collision>
+      <origin
+        xyz="0 0 0"
+        rpy="0 0 0" />
+      <geometry>
+        <mesh
+          filename="${mesh_prefix}/models/so_100_arm_5dof/meshes/Wrist_Pitch_Roll.STL" />
       </geometry>
     </collision>
@@ -326,19 +302,19 @@
       <geometry>
         <mesh
-          filename="package://gimbal_mani/models/so_100_arm_5dof/meshes/Fixed_Gripper.STL" />
-      </geometry>
-      <material
-        name="">
-        <color
-          rgba="0.792156862745098 0.819607843137255 0.933333333333333 1" />
-      </material>
-    </visual>
-    <collision>
-      <origin
-        xyz="0 0 0"
-        rpy="0 0 0" />
-      <geometry>
-        <mesh
-          filename="package://gimbal_mani/models/so_100_arm_5dof/meshes/Fixed_Gripper.STL" />
+          filename="${mesh_prefix}/models/so_100_arm_5dof/meshes/Fixed_Gripper.STL" />
+      </geometry>
+      <material
+        name="">
+        <color
+          rgba="0.792156862745098 0.819607843137255 0.933333333333333 1" />
+      </material>
+    </visual>
+    <collision>
+      <origin
+        xyz="0 0 0"
+        rpy="0 0 0" />
+      <geometry>
+        <mesh
+          filename="${mesh_prefix}/models/so_100_arm_5dof/meshes/Fixed_Gripper.STL" />
       </geometry>
     </collision>
@@ -350,5 +326,5 @@
       <geometry>
         <mesh
-          filename="package://gimbal_mani/models/gimbal/meshes/gimbal_mount.STL"
+          filename="${mesh_prefix}/models/gimbal/meshes/gimbal_mount.STL"
           scale="0.001 0.001 0.001"/>
       </geometry>
@@ -399,19 +375,19 @@
       <geometry>
         <mesh
-          filename="package://gimbal_mani/models/so_100_arm_5dof/meshes/Moving_Jaw.STL" />
-      </geometry>
-      <material
-        name="">
-        <color
-          rgba="0.792156862745098 0.819607843137255 0.933333333333333 1" />
-      </material>
-    </visual>
-    <collision>
-      <origin
-        xyz="0 0 0"
-        rpy="0 0 0" />
-      <geometry>
-        <mesh
-          filename="package://gimbal_mani/models/so_100_arm_5dof/meshes/Moving_Jaw.STL" />
+          filename="${mesh_prefix}/models/so_100_arm_5dof/meshes/Moving_Jaw.STL" />
+      </geometry>
+      <material
+        name="">
+        <color
+          rgba="0.792156862745098 0.819607843137255 0.933333333333333 1" />
+      </material>
+    </visual>
+    <collision>
+      <origin
+        xyz="0 0 0"
+        rpy="0 0 0" />
+      <geometry>
+        <mesh
+          filename="${mesh_prefix}/models/so_100_arm_5dof/meshes/Moving_Jaw.STL" />
       </geometry>
     </collision>

Commit message: 동작 범위 수정

File: urdf/so_100_arm_5dof.urdf.xacro (robot description, xacro)
@@ -104,5 +104,5 @@
   <joint
     name="Shoulder_Rotation"
-    type="continuous">
+    type="revolute">
     <origin
       xyz="0 -0.0452 0.0165"
@@ -114,5 +114,5 @@
     <axis
       xyz="0 1 0" />
-    <limit lower="-3.14" upper="3.14" effort="10" velocity="2.0"/>
+    <limit lower="-1.5708" upper="1.5708" effort="10" velocity="2.0"/>
   </joint>
   <link
@@ -158,5 +158,5 @@
   <joint
     name="Shoulder_Pitch"
-    type="continuous">
+    type="revolute">
     <origin
       xyz="0 0.1025 0.0306"
@@ -168,5 +168,5 @@
     <axis
       xyz="1 0 0" />
-    <limit lower="-3.14" upper="3.14" effort="10" velocity="2.0"/>
+    <limit lower="-1.5708" upper="1.5708" effort="10" velocity="2.0"/>
   </joint>
   <link
@@ -212,5 +212,5 @@
   <joint
     name="Elbow"
-    type="continuous">
+    type="revolute">
     <origin
       xyz="0 0.11257 0.028"
@@ -222,5 +222,5 @@
     <axis
       xyz="1 0 0" />
-    <limit lower="-3.14" upper="3.14" effort="10" velocity="2.0"/>
+    <limit lower="-1.5708" upper="1.5708" effort="10" velocity="2.0"/>
   </joint>
   <link
@@ -266,5 +266,5 @@
   <joint
     name="Wrist_Pitch"
-    type="continuous">
+    type="revolute">
     <origin
       xyz="0 0.0052 0.1349"
@@ -276,5 +276,5 @@
     <axis
       xyz="1 0 0" />
-    <limit lower="-3.14" upper="3.14" effort="10" velocity="2.0"/>
+    <limit lower="-3.1416" upper="0.0" effort="10" velocity="2.0"/>
   </joint>
   <link
@@ -317,7 +317,13 @@
       </geometry>
     </collision>
-  </link>
-  <link
-    name="gimbal_mount_link">
+	  </link>
+	  <link name="gripper_grasp_frame"/>
+	  <joint name="fixed_gripper_to_grasp_frame" type="fixed">
+	    <parent link="Fixed_Gripper"/>
+	    <child link="gripper_grasp_frame"/>
+	    <origin xyz="-0.010 -0.055 -0.030" rpy="0 0 0"/>
+	  </joint>
+	  <link
+	    name="gimbal_mount_link">
     <visual>
       <origin xyz="0 0 0" rpy="0 0 0"/>
@@ -339,5 +345,5 @@
   <joint
     name="Wrist_Roll"
-    type="continuous">
+    type="revolute">
     <origin
       xyz="0 -0.0601 0"
@@ -349,5 +355,5 @@
     <axis
       xyz="0 1 0" />
-    <limit lower="-3.14" upper="3.14" effort="10" velocity="2.0"/>
+    <limit lower="-0.001" upper="0.001" effort="10" velocity="2.0"/>
   </joint>
   <link
@@ -393,5 +399,5 @@
   <joint
     name="Gripper"
-    type="continuous">
+    type="revolute">
     <origin
       xyz="-0.0202 -0.0244 0"
@@ -403,5 +409,5 @@
     <axis
       xyz="0 0 1" />
-    <limit lower="-3.14" upper="3.14" effort="10" velocity="2.0"/>
+    <limit lower="0.0" upper="1.5" effort="10" velocity="2.0"/>
   </joint>
 </robot>

Commit message: 그리퍼에 마찰 추가

File: urdf/so_100_arm_5dof.urdf.xacro (robot description, xacro)
@@ -5,5 +5,5 @@
 <robot
   name="so_100_arm" xmlns:xacro="http://www.ros.org/wiki/xacro">
-  <xacro:arg name="mesh_prefix" default=""/>
+  <xacro:arg name="mesh_prefix" default="package://gimbal_mani"/>
 <!--
   <link name="world"/>
@@ -317,4 +317,10 @@
       </geometry>
     </collision>
+    <collision name="fixed_gripper_contact_pad">
+      <origin xyz="0.0133 -0.0625 0" rpy="0 0 0"/>
+      <geometry>
+        <box size="0.001 0.035 0.025"/>
+      </geometry>
+    </collision>
 	  </link>
 	  <link name="gripper_grasp_frame"/>
@@ -330,5 +336,5 @@
       <geometry>
         <mesh
-          filename="${mesh_prefix}/models/gimbal/meshes/gimbal_mount.STL"
+          filename="${mesh_prefix}/models/gimbal/meshes/gimbal_mount.stl"
           scale="0.001 0.001 0.001"/>
       </geometry>
@@ -396,4 +402,10 @@
       </geometry>
     </collision>
+    <collision name="moving_jaw_contact_pad">
+      <origin xyz="-0.0083 -0.0381 0" rpy="0 0 0"/>
+      <geometry>
+        <box size="0.001 0.035 0.025"/>
+      </geometry>
+    </collision>
   </link>
   <joint
@@ -411,3 +423,19 @@
     <limit lower="0.0" upper="1.5" effort="10" velocity="2.0"/>
   </joint>
+  <gazebo reference="Fixed_Gripper">
+    <mu1>1.5</mu1>
+    <mu2>1.5</mu2>
+    <kp>100000.0</kp>
+    <kd>10.0</kd>
+    <maxVel>0.001</maxVel>
+    <minDepth>0.0001</minDepth>
+  </gazebo>
+  <gazebo reference="Moving_Jaw">
+    <mu1>1.5</mu1>
+    <mu2>1.5</mu2>
+    <kp>100000.0</kp>
+    <kd>10.0</kd>
+    <maxVel>0.001</maxVel>
+    <minDepth>0.0001</minDepth>
+  </gazebo>
 </robot>
